File: schematics/schematics/schematics (copia).kicad_pcb (KiCad board)
At the start: 2 copper layers, 63.5 x 64.8 mm, 35 parts, among them J1 Conn_01x02, J2 Conn_01x03, J4 Conn_01x02, K1 SANYOU_SRD_Form_C, SW2 SW_Push, U1 ESP32-WROVER, U2 RC522, U3 AS608, U4 MT3608_PCB, U5 AMS1117

Commit message: .
Parts:
- removed C7: 47uF, Capacitor_SMD:C_0603_1608Metric_Pad1.05x0.95mm_HandSolder
- removed C8: 100uF, Capacitor_SMD:C_0603_1608Metric_Pad1.05x0.95mm_HandSolder
- removed D10: 1N5406, Diode_SMD:D_1206_3216Metric_Pad1.42x1.75mm_HandSolder
- removed J4: Conn_01x02, Connector_JST:JST_EH_B2B-EH-A_1x02_P2.50mm_Vertical
- removed U4: MT3608_PCB, mt3608:mt3608pcb
- removed U5: AMS1117, Package_TO_SOT_SMD:SOT-223-3_TabPin2
- added BTR1: Conn_01x02, Connector_JST:JST_EH_B2B-EH-A_1x02_P2.50mm_Vertical, F.Cu at (138.7, 111.5)
- added BTR2: Conn_01x02, Connector_JST:JST_EH_B2B-EH-A_1x02_P2.50mm_Vertical, F.Cu at (127.8, 111.5)
- added TP4056-1: , TP4056:TP4056-18650, F.Cu at (119.9, 86.4)
- added TP4056-2: , TP4056:TP4056-18650, F.Cu at (99.6, 113.3)
- added U3V12F12: , Connector_PinHeader_2.00mm:PinHeader_1x03_P2.00mm_Vertical, F.Cu at (91.2, 108.0)
- R2, R3, R4, R5, R6, R7: value 100 -> 220
Routing:
- net GND: track 349.7 -> 300.7 mm
- net Net-(TP4056-1-Pad1): track 0.00 -> 32.9 mm
- net /Potencia/BTR2+: track 0.00 -> 32.0 mm
- net /Potencia/BTR2-: track 0.00 -> 31.5 mm
- net /Cerradura/12v: track 50.2 -> 75.0 mm
- net Net-(C8-Pad1): track 24.4 -> 0.00 mm
- net /Potencia/BTR1+: track 0.00 -> 24.4 mm
- net /Potencia/BTR1-: track 0.00 -> 15.7 mm
- net Net-(TP4056-1-Pad2): track 0.00 -> 12.8 mm
- net Net-(D10-Pad2): track 7.08 -> 0.00 mm
- net /AS608/3v3: track 162.0 -> 161.0 mm
- removed copper zone on B.Cu, net GND
Other:
- board size 63.5 x 64.8 mm -> 63.5 x 75.2 mm
