File: schematics/schematics/AS608.sch (KiCad schematic (older format))
At the start: 1 part, among them U3 AS608

Commit message: .
Parts:
- U3: LCSC (none) -> C144395
Changed lines of the file:
@@
 F 2 "Connector_JST:JST_EH_B4B-EH-A_1x04_P2.50mm_Vertical" H 5100 3150 50  0001 C CNN
 F 3 "" H 5100 3150 50  0001 C CNN
+F 4 "C144395" H 5350 3100 50  0001 C CNN "LCSC"
 	1    5350 3100
 	1    0    0    -1
