File: schematics/schematics/RC522.sch (KiCad schematic (older format))
At the start: 1 part, among them U2 RC522

Commit message: .
Parts:
- U2: footprint ESP32-WROVER-I:RC522 -> Connector_JST:JST_EH_B8B-EH-A_1x08_P2.50mm_Vertical
Changed lines of the file:
@@
 F 0 "U2" H 4625 4115 50  0000 C CNN
 F 1 "RC522" H 4625 4024 50  0000 C CNN
-F 2 "ESP32-WROVER-I:RC522" H 4600 4100 50  0001 C CNN
+F 2 "Connector_JST:JST_EH_B8B-EH-A_1x08_P2.50mm_Vertical" H 4600 4100 50  0001 C CNN
 F 3 "" H 4600 4100 50  0001 C CNN
 	1    4250 3350

Commit message: .
Parts:
- U2: LCSC (none) -> C161875
Changed lines of the file:
@@
 F 2 "Connector_JST:JST_EH_B8B-EH-A_1x08_P2.50mm_Vertical" H 4600 4100 50  0001 C CNN
 F 3 "" H 4600 4100 50  0001 C CNN
+F 4 "C161875" H 4250 3350 50  0001 C CNN "LCSC"
 	1    4250 3350
 	1    0    0    -1
