File: schematics/schematics/Cerradura.sch (KiCad schematic (older format))
At the start: 4 parts, among them J1 Conn_01x02, K1 SANYOU_SRD_Form_C

Commit message: .
Parts:
- D7, D8: footprint Diode_THT:D_DO-41_SOD81_P7.62mm_Horizontal -> Diode_SMD:D_1206_3216Metric_Pad1.42x1.75mm_HandSolder
Changed lines of the file:
@@
 F 0 "D7" V 4354 4129 50  0000 L CNN
 F 1 "D" V 4445 4129 50  0000 L CNN
-F 2 "Diode_THT:D_DO-41_SOD81_P7.62mm_Horizontal" H 4400 4050 50  0001 C CNN
+F 2 "Diode_SMD:D_1206_3216Metric_Pad1.42x1.75mm_HandSolder" H 4400 4050 50  0001 C CNN
 F 3 "~" H 4400 4050 50  0001 C CNN
 	1    4400 4050
@@
 F 0 "D8" H 4000 3016 50  0000 C CNN
 F 1 "D" H 4000 2925 50  0000 C CNN
-F 2 "Diode_THT:D_DO-41_SOD81_P7.62mm_Horizontal" H 4000 2800 50  0001 C CNN
+F 2 "Diode_SMD:D_1206_3216Metric_Pad1.42x1.75mm_HandSolder" H 4000 2800 50  0001 C CNN
 F 3 "~" H 4000 2800 50  0001 C CNN
 	1    4000 2800

Commit message: .
Parts:
- renumbered J1 to Cerradura1
Changed lines of the file:
@@
 Connection ~ 4400 4200
 $Comp
-L Connector_Generic:Conn_01x02 J1
+L Connector_Generic:Conn_01x02 Cerradura1
 U 1 1 61954441
 P 4950 3850
-F 0 "J1" H 5030 3842 50  0000 L CNN
+F 0 "Cerradura1" H 5030 3842 50  0000 L CNN
 F 1 "Conn_01x02" H 5030 3751 50  0000 L CNN
 F 2 "Connector_JST:JST_EH_B2B-EH-A_1x02_P2.50mm_Vertical" H 4950 3850 50  0001 C CNN

Commit message: .
Parts:
- Cerradura1: LCSC (none) -> C158012
Changed lines of the file:
@@
 F 2 "Connector_JST:JST_EH_B2B-EH-A_1x02_P2.50mm_Vertical" H 4950 3850 50  0001 C CNN
 F 3 "~" H 4950 3850 50  0001 C CNN
+F 4 "C158012" H 4950 3850 50  0001 C CNN "LCSC"
 	1    4950 3850
 	1    0    0    -1

Commit message: .
Parts:
- D7, D8: footprint Diode_SMD:D_1206_3216Metric_Pad1.42x1.75mm_HandSolder -> Diode_SMD:D_SOD-123; LCSC (none) -> C162734
- K1: LCSC (none) -> C24585
Changed lines of the file:
@@
 F 2 "Relay_THT:Relay_SPDT_SANYOU_SRD_Series_Form_C" H 4450 3500 50  0001 L CNN
 F 3 "http://www.sanyourelay.ca/public/products/pdf/SRD.pdf" H 4000 3550 50  0001 C CNN
+F 4 "C24585" V 4000 3550 50  0001 C CNN "LCSC"
 	1    4000 3550
 	0    1    1    0
@@
 F 0 "D7" V 4354 4129 50  0000 L CNN
 F 1 "D" V 4445 4129 50  0000 L CNN
-F 2 "Diode_SMD:D_1206_3216Metric_Pad1.42x1.75mm_HandSolder" H 4400 4050 50  0001 C CNN
+F 2 "Diode_SMD:D_SOD-123" H 4400 4050 50  0001 C CNN
 F 3 "~" H 4400 4050 50  0001 C CNN
+F 4 "C162734" V 4400 4050 50  0001 C CNN "LCSC"
 	1    4400 4050
 	0    1    1    0
@@
 F 0 "D8" H 4000 3016 50  0000 C CNN
 F 1 "D" H 4000 2925 50  0000 C CNN
-F 2 "Diode_SMD:D_1206_3216Metric_Pad1.42x1.75mm_HandSolder" H 4000 2800 50  0001 C CNN
+F 2 "Diode_SMD:D_SOD-123" H 4000 2800 50  0001 C CNN
 F 3 "~" H 4000 2800 50  0001 C CNN
+F 4 "C162734" H 4000 2800 50  0001 C CNN "LCSC"
 	1    4000 2800
 	1    0    0    -1
