File: schematics/schematics/ESP32.sch (KiCad schematic (older format))
At the start: 19 parts, among them U1 ESP32-WROVER

Commit message: .
Parts:
- D1, D2, D3, D4, D5, D6: footprint LED_THT:LED_D3.0mm -> LED_SMD:LED_0603_1608Metric_Pad1.05x0.95mm_HandSolder
- R2, R3, R4, R5, R6, R7: value 220 -> 100
Changed lines of the file:
@@
 AR Path="/618FDA94/61995CB9" Ref="R2"  Part="1"
 F 0 "R2" H 4520 5196 50  0000 L CNN
-F 1 "220" H 4520 5105 50  0000 L CNN
+F 1 "100" H 4520 5105 50  0000 L CNN
 F 2 "Resistor_SMD:R_1206_3216Metric_Pad1.42x1.75mm_HandSolder" V 4380 5150 50  0001 C CNN
 F 3 "~" H 4450 5150 50  0001 C CNN
@@
 F 0 "D1" V 4489 5383 50  0000 R CNN
 F 1 "LED" V 4398 5383 50  0000 R CNN
-F 2 "LED_THT:LED_D3.0mm" H 4450 5500 50  0001 C CNN
+F 2 "LED_SMD:LED_0603_1608Metric_Pad1.05x0.95mm_HandSolder" H 4450 5500 50  0001 C CNN
 F 3 "~" H 4450 5500 50  0001 C CNN
 	1    4450 5500
@@
 AR Path="/618FDA94/619B051C" Ref="R3"  Part="1"
 F 0 "R3" H 4220 5196 50  0000 L CNN
-F 1 "220" H 4220 5105 50  0000 L CNN
+F 1 "100" H 4220 5105 50  0000 L CNN
 F 2 "Resistor_SMD:R_1206_3216Metric_Pad1.42x1.75mm_HandSolder" V 4080 5150 50  0001 C CNN
 F 3 "~" H 4150 5150 50  0001 C CNN
@@
 F 0 "D2" V 4189 5383 50  0000 R CNN
 F 1 "LED" V 4098 5383 50  0000 R CNN
-F 2 "LED_THT:LED_D3.0mm" H 4150 5500 50  0001 C CNN
+F 2 "LED_SMD:LED_0603_1608Metric_Pad1.05x0.95mm_HandSolder" H 4150 5500 50  0001 C CNN
 F 3 "~" H 4150 5500 50  0001 C CNN
 	1    4150 5500
@@
 AR Path="/618FDA94/619B18F8" Ref="R4"  Part="1"
 F 0 "R4" H 3920 5196 50  0000 L CNN
-F 1 "220" H 3920 5105 50  0000 L CNN
+F 1 "100" H 3920 5105 50  0000 L CNN
 F 2 "Resistor_SMD:R_1206_3216Metric_Pad1.42x1.75mm_HandSolder" V 3780 5150 50  0001 C CNN
 F 3 "~" H 3850 5150 50  0001 C CNN
@@
 F 0 "D3" V 3889 5383 50  0000 R CNN
 F 1 "LED" V 3798 5383 50  0000 R CNN
-F 2 "LED_THT:LED_D3.0mm" H 3850 5500 50  0001 C CNN
+F 2 "LED_SMD:LED_0603_1608Metric_Pad1.05x0.95mm_HandSolder" H 3850 5500 50  0001 C CNN
 F 3 "~" H 3850 5500 50  0001 C CNN
 	1    3850 5500
@@
 AR Path="/618FDA94/61974CB1" Ref="R6"  Part="1"
 F 0 "R6" H 5120 5196 50  0000 L CNN
-F 1 "220" H 5120 5105 50  0000 L CNN
+F 1 "100" H 5120 5105 50  0000 L CNN
 F 2 "Resistor_SMD:R_1206_3216Metric_Pad1.42x1.75mm_HandSolder" V 4980 5150 50  0001 C CNN
 F 3 "~" H 5050 5150 50  0001 C CNN
@@
 F 0 "D5" V 5089 5383 50  0000 R CNN
 F 1 "LED" V 4998 5383 50  0000 R CNN
-F 2 "LED_THT:LED_D3.0mm" H 5050 5500 50  0001 C CNN
+F 2 "LED_SMD:LED_0603_1608Metric_Pad1.05x0.95mm_HandSolder" H 5050 5500 50  0001 C CNN
 F 3 "~" H 5050 5500 50  0001 C CNN
 	1    5050 5500
@@
 AR Path="/618FDA94/61974CC5" Ref="R5"  Part="1"
 F 0 "R5" H 4820 5196 50  0000 L CNN
-F 1 "220" H 4820 5105 50  0000 L CNN
+F 1 "100" H 4820 5105 50  0000 L CNN
 F 2 "Resistor_SMD:R_1206_3216Metric_Pad1.42x1.75mm_HandSolder" V 4680 5150 50  0001 C CNN
 F 3 "~" H 4750 5150 50  0001 C CNN
@@
 F 0 "D4" V 4789 5383 50  0000 R CNN
 F 1 "LED" V 4698 5383 50  0000 R CNN
-F 2 "LED_THT:LED_D3.0mm" H 4750 5500 50  0001 C CNN
+F 2 "LED_SMD:LED_0603_1608Metric_Pad1.05x0.95mm_HandSolder" H 4750 5500 50  0001 C CNN
 F 3 "~" H 4750 5500 50  0001 C CNN
 	1    4750 5500
@@
 AR Path="/618FDA94/619A1451" Ref="R7"  Part="1"
 F 0 "R7" H 5420 5196 50  0000 L CNN
-F 1 "220" H 5420 5105 50  0000 L CNN
+F 1 "100" H 5420 5105 50  0000 L CNN
 F 2 "Resistor_SMD:R_1206_3216Metric_Pad1.42x1.75mm_HandSolder" V 5280 5150 50  0001 C CNN
 F 3 "~" H 5350 5150 50  0001 C CNN
@@
 F 0 "D6" V 5389 5383 50  0000 R CNN
 F 1 "LED" V 5298 5383 50  0000 R CNN
-F 2 "LED_THT:LED_D3.0mm" H 5350 5500 50  0001 C CNN
+F 2 "LED_SMD:LED_0603_1608Metric_Pad1.05x0.95mm_HandSolder" H 5350 5500 50  0001 C CNN
 F 3 "~" H 5350 5500 50  0001 C CNN
 	1    5350 5500

Commit message: .
Parts:
- C4: value C -> 100 pF
Changed lines of the file:
@@
 P 5450 3350
 F 0 "C4" H 5565 3396 50  0000 L CNN
-F 1 "C" H 5565 3305 50  0000 L CNN
+F 1 "100 pF" H 5565 3305 50  0000 L CNN
 F 2 "Capacitor_SMD:C_0603_1608Metric_Pad1.05x0.95mm_HandSolder" H 5488 3200 50  0001 C CNN
 F 3 "~" H 5450 3350 50  0001 C CNN

Commit message: .
Parts:
- C1: LCSC (none) -> C271438
- C2: LCSC (none) -> C96446
- C4: LCSC (none) -> C0603
- D1: value LED -> On; LCSC (none) -> C189306
- D2: value LED -> Wifi; LCSC (none) -> C138547
- D3: value LED -> Open; LCSC (none) -> C118330
- D4: value LED -> lvl1; LCSC (none) -> C375447
- D5: value LED -> lvl2; LCSC (none) -> C138546
- D6: value LED -> lvl3; LCSC (none) -> C118330
- R1: LCSC (none) -> C17902
- R2, R3, R4, R5, R6, R7: LCSC (none) -> C17408
- U1: LCSC (none) -> C529591
Changed lines of the file:
@@
 F 2 "Capacitor_SMD:C_0603_1608Metric_Pad1.05x0.95mm_HandSolder" H 4138 3250 50  0001 C CNN
 F 3 "~" H 4100 3400 50  0001 C CNN
+F 4 "C271438" H 4100 3400 50  0001 C CNN "LCSC"
 	1    4100 3400
 	1    0    0    -1
@@
 F 2 "Capacitor_SMD:C_0603_1608Metric_Pad1.05x0.95mm_HandSolder" H 3738 3250 50  0001 C CNN
 F 3 "~" H 3700 3400 50  0001 C CNN
+F 4 "C96446" H 3700 3400 50  0001 C CNN "LCSC"
 	1    3700 3400
 	1    0    0    -1
@@
 F 2 "Resistor_SMD:R_1206_3216Metric_Pad1.42x1.75mm_HandSolder" V 4830 3900 50  0001 C CNN
 F 3 "~" H 4900 3900 50  0001 C CNN
+F 4 "C17902" H 4900 3900 50  0001 C CNN "LCSC"
 	1    4900 3900
 	1    0    0    -1
@@
 F 2 "Resistor_SMD:R_1206_3216Metric_Pad1.42x1.75mm_HandSolder" V 4380 5150 50  0001 C CNN
 F 3 "~" H 4450 5150 50  0001 C CNN
+F 4 "C17408" H 4450 5150 50  0001 C CNN "LCSC"
 	1    4450 5150
 	1    0    0    -1
-$EndComp
-$Comp
-L Device:LED D?
-U 1 1 61995CBF
-P 4450 5500
-AR Path="/61995CBF" Ref="D?"  Part="1"
-AR Path="/618FDA94/61995CBF" Ref="D1"  Part="1"
-F 0 "D1" V 4489 5383 50  0000 R CNN
-F 1 "LED" V 4398 5383 50  0000 R CNN
-F 2 "LED_SMD:LED_0603_1608Metric_Pad1.05x0.95mm_HandSolder" H 4450 5500 50  0001 C CNN
-F 3 "~" H 4450 5500 50  0001 C CNN
-	1    4450 5500
-	0    -1   -1   0
 $EndComp
 Wire Wire Line
@@
 F 2 "Resistor_SMD:R_1206_3216Metric_Pad1.42x1.75mm_HandSolder" V 4080 5150 50  0001 C CNN
 F 3 "~" H 4150 5150 50  0001 C CNN
+F 4 "C17408" H 4150 5150 50  0001 C CNN "LCSC"
 	1    4150 5150
 	1    0    0    -1
-$EndComp
-$Comp
-L Device:LED D?
-U 1 1 619B0522
-P 4150 5500
-AR Path="/619B0522" Ref="D?"  Part="1"
-AR Path="/618FDA94/619B0522" Ref="D2"  Part="1"
-F 0 "D2" V 4189 5383 50  0000 R CNN
-F 1 "LED" V 4098 5383 50  0000 R CNN
-F 2 "LED_SMD:LED_0603_1608Metric_Pad1.05x0.95mm_HandSolder" H 4150 5500 50  0001 C CNN
-F 3 "~" H 4150 5500 50  0001 C CNN
-	1    4150 5500
-	0    -1   -1   0
 $EndComp
 Wire Wire Line
@@
 F 2 "Resistor_SMD:R_1206_3216Metric_Pad1.42x1.75mm_HandSolder" V 3780 5150 50  0001 C CNN
 F 3 "~" H 3850 5150 50  0001 C CNN
+F 4 "C17408" H 3850 5150 50  0001 C CNN "LCSC"
 	1    3850 5150
 	1    0    0    -1
-$EndComp
-$Comp
-L Device:LED D?
-U 1 1 619B18FE
-P 3850 5500
-AR Path="/619B18FE" Ref="D?"  Part="1"
-AR Path="/618FDA94/619B18FE" Ref="D3"  Part="1"
-F 0 "D3" V 3889 5383 50  0000 R CNN
-F 1 "LED" V 3798 5383 50  0000 R CNN
-F 2 "LED_SMD:LED_0603_1608Metric_Pad1.05x0.95mm_HandSolder" H 3850 5500 50  0001 C CNN
-F 3 "~" H 3850 5500 50  0001 C CNN
-	1    3850 5500
-	0    -1   -1   0
 $EndComp
 Wire Wire Line
@@
 F 2 "ESP32-WROVER-I:XCVR_ESP32-WROVER-I" H 7350 3850 60  0001 C CNN
 F 3 "" H 7350 3850 60  0001 C CNN
+F 4 "C529591" H 6900 4150 50  0001 C CNN "LCSC"
 	1    6900 4150
 	1    0    0    -1
@@
 F 2 "Resistor_SMD:R_1206_3216Metric_Pad1.42x1.75mm_HandSolder" V 4980 5150 50  0001 C CNN
 F 3 "~" H 5050 5150 50  0001 C CNN
+F 4 "C17408" H 5050 5150 50  0001 C CNN "LCSC"
 	1    5050 5150
 	1    0    0    -1
-$EndComp
-$Comp
-L Device:LED D?
-U 1 1 61974CB7
-P 5050 5500
-AR Path="/61974CB7" Ref="D?"  Part="1"
-AR Path="/618FDA94/61974CB7" Ref="D5"  Part="1"
-F 0 "D5" V 5089 5383 50  0000 R CNN
-F 1 "LED" V 4998 5383 50  0000 R CNN
-F 2 "LED_SMD:LED_0603_1608Metric_Pad1.05x0.95mm_HandSolder" H 5050 5500 50  0001 C CNN
-F 3 "~" H 5050 5500 50  0001 C CNN
-	1    5050 5500
-	0    -1   -1   0
 $EndComp
 Wire Wire Line
@@
 	1    0    0    -1
 $EndComp
-$Comp
-L Device:R R?
-U 1 1 61974CC5
-P 4750 5150
-AR Path="/61974CC5" Ref="R?"  Part="1"
-AR Path="/618FDA94/61974CC5" Ref="R5"  Part="1"
-F 0 "R5" H 4820 5196 50  0000 L CNN
-F 1 "100" H 4820 5105 50  0000 L CNN
-F 2 "Resistor_SMD:R_1206_3216Metric_Pad1.42x1.75mm_HandSolder" V 4680 5150 50  0001 C CNN
-F 3 "~" H 4750 5150 50  0001 C CNN
-	1    4750 5150
-	1    0    0    -1
-$EndComp
-$Comp
-L Device:LED D?
-U 1 1 61974CCB
-P 4750 5500
-AR Path="/61974CCB" Ref="D?"  Part="1"
-AR Path="/618FDA94/61974CCB" Ref="D4"  Part="1"
-F 0 "D4" V 4789 5383 50  0000 R CNN
-F 1 "LED" V 4698 5383 50  0000 R CNN
-F 2 "LED_SMD:LED_0603_1608Metric_Pad1.05x0.95mm_HandSolder" H 4750 5500 50  0001 C CNN
-F 3 "~" H 4750 5500 50  0001 C CNN
-	1    4750 5500
-	0    -1   -1   0
-$EndComp
 Wire Wire Line
 	4750 4600 6000 4600
@@
 F 2 "Resistor_SMD:R_1206_3216Metric_Pad1.42x1.75mm_HandSolder" V 5280 5150 50  0001 C CNN
 F 3 "~" H 5350 5150 50  0001 C CNN
+F 4 "C17408" H 5350 5150 50  0001 C CNN "LCSC"
 	1    5350 5150
 	1    0    0    -1
-$EndComp
-$Comp
-L Device:LED D?
-U 1 1 619A1457
-P 5350 5500
-AR Path="/619A1457" Ref="D?"  Part="1"
-AR Path="/618FDA94/619A1457" Ref="D6"  Part="1"
-F 0 "D6" V 5389 5383 50  0000 R CNN
-F 1 "LED" V 5298 5383 50  0000 R CNN
-F 2 "LED_SMD:LED_0603_1608Metric_Pad1.05x0.95mm_HandSolder" H 5350 5500 50  0001 C CNN
-F 3 "~" H 5350 5500 50  0001 C CNN
-	1    5350 5500
-	0    -1   -1   0
 $EndComp
 Wire Wire Line
@@
 F 2 "Capacitor_SMD:C_0603_1608Metric_Pad1.05x0.95mm_HandSolder" H 5488 3200 50  0001 C CNN
 F 3 "~" H 5450 3350 50  0001 C CNN
+F 4 "C0603" H 5450 3350 50  0001 C CNN "LCSC"
 	1    5450 3350
 	1    0    0    -1
@@
 Wire Wire Line
 	4900 3600 6000 3600
+$Comp
+L Device:R R?
+U 1 1 61974CC5
+P 4750 5150
+AR Path="/61974CC5" Ref="R?"  Part="1"
+AR Path="/618FDA94/61974CC5" Ref="R5"  Part="1"
+F 0 "R5" H 4820 5196 50  0000 L CNN
+F 1 "100" H 4820 5105 50  0000 L CNN
+F 2 "Resistor_SMD:R_1206_3216Metric_Pad1.42x1.75mm_HandSolder" V 4680 5150 50  0001 C CNN
+F 3 "~" H 4750 5150 50  0001 C CNN
+F 4 "C17408" H 4750 5150 50  0001 C CNN "LCSC"
+	1    4750 5150
+	1    0    0    -1
+$EndComp
+$Comp
+L Device:LED D?
+U 1 1 619A1457
+P 5350 5500
+AR Path="/619A1457" Ref="D?"  Part="1"
+AR Path="/618FDA94/619A1457" Ref="D6"  Part="1"
+F 0 "D6" V 5389 5383 50  0000 R CNN
+F 1 "lvl3" V 5298 5383 50  0000 R CNN
+F 2 "LED_SMD:LED_0603_1608Metric_Pad1.05x0.95mm_HandSolder" H 5350 5500 50  0001 C CNN
+F 3 "~" H 5350 5500 50  0001 C CNN
+F 4 "C118330" V 5350 5500 50  0001 C CNN "LCSC"
+	1    5350 5500
+	0    -1   -1   0
+$EndComp
+$Comp
+L Device:LED D?
+U 1 1 61974CB7
+P 5050 5500
+AR Path="/61974CB7" Ref="D?"  Part="1"
+AR Path="/618FDA94/61974CB7" Ref="D5"  Part="1"
+F 0 "D5" V 5089 5383 50  0000 R CNN
+F 1 "lvl2" V 4998 5383 50  0000 R CNN
+F 2 "LED_SMD:LED_0603_1608Metric_Pad1.05x0.95mm_HandSolder" H 5050 5500 50  0001 C CNN
+F 3 "~" H 5050 5500 50  0001 C CNN
+F 4 "C138546" V 5050 5500 50  0001 C CNN "LCSC"
+	1    5050 5500
+	0    -1   -1   0
+$EndComp
+$Comp
+L Device:LED D?
+U 1 1 61974CCB
+P 4750 5500
+AR Path="/61974CCB" Ref="D?"  Part="1"
+AR Path="/618FDA94/61974CCB" Ref="D4"  Part="1"
+F 0 "D4" V 4789 5383 50  0000 R CNN
+F 1 "lvl1" V 4698 5383 50  0000 R CNN
+F 2 "LED_SMD:LED_0603_1608Metric_Pad1.05x0.95mm_HandSolder" H 4750 5500 50  0001 C CNN
+F 3 "~" H 4750 5500 50  0001 C CNN
+F 4 "C375447" V 4750 5500 50  0001 C CNN "LCSC"
+	1    4750 5500
+	0    -1   -1   0
+$EndComp
+$Comp
+L Device:LED D?
+U 1 1 619B0522
+P 4150 5500
+AR Path="/619B0522" Ref="D?"  Part="1"
+AR Path="/618FDA94/619B0522" Ref="D2"  Part="1"
+F 0 "D2" V 4189 5383 50  0000 R CNN
+F 1 "Wifi" V 4098 5383 50  0000 R CNN
+F 2 "LED_SMD:LED_0603_1608Metric_Pad1.05x0.95mm_HandSolder" H 4150 5500 50  0001 C CNN
+F 3 "~" H 4150 5500 50  0001 C CNN
+F 4 "C138547" V 4150 5500 50  0001 C CNN "LCSC"
+	1    4150 5500
+	0    -1   -1   0
+$EndComp
+$Comp
+L Device:LED D?
+U 1 1 61995CBF
+P 4450 5500
+AR Path="/61995CBF" Ref="D?"  Part="1"
+AR Path="/618FDA94/61995CBF" Ref="D1"  Part="1"
+F 0 "D1" V 4489 5383 50  0000 R CNN
+F 1 "On" V 4398 5383 50  0000 R CNN
+F 2 "LED_SMD:LED_0603_1608Metric_Pad1.05x0.95mm_HandSolder" H 4450 5500 50  0001 C CNN
+F 3 "~" H 4450 5500 50  0001 C CNN
+F 4 "C189306" V 4450 5500 50  0001 C CNN "LCSC"
+	1    4450 5500
+	0    -1   -1   0
+$EndComp
+$Comp
+L Device:LED D?
+U 1 1 619B18FE
+P 3850 5500
+AR Path="/619B18FE" Ref="D?"  Part="1"
+AR Path="/618FDA94/619B18FE" Ref="D3"  Part="1"
+F 0 "D3" V 3889 5383 50  0000 R CNN
+F 1 "Open" V 3798 5383 50  0000 R CNN
+F 2 "LED_SMD:LED_0603_1608Metric_Pad1.05x0.95mm_HandSolder" H 3850 5500 50  0001 C CNN
+F 3 "~" H 3850 5500 50  0001 C CNN
+F 4 "C118330" V 3850 5500 50  0001 C CNN "LCSC"
+	1    3850 5500
+	0    -1   -1   0
+$EndComp
 $EndSCHEMATC

Commit message: .
Parts:
- C1: footprint Capacitor_SMD:C_0603_1608Metric_Pad1.05x0.95mm_HandSolder -> Capacitor_THT:CP_Radial_D4.0mm_P2.00mm
- C3: footprint Capacitor_SMD:C_0603_1608Metric_Pad1.05x0.95mm_HandSolder -> Capacitor_THT:CP_Radial_D5.0mm_P2.50mm
- C4: LCSC C0603 -> C44567
- D2: LCSC C138547 -> C375447
- RESET1: footprint Button_Switch_THT:SW_PUSH_6mm -> RC522:boton
Connections:
- net 3v3: now also R1.1; no longer C3.1, RESET1.2
- net GND: now also C3.2, RESET1.1; no longer R1.2
- new net: C3.1, R1.2, RESET1.2, U1.3 (EN)
Other:
- moved on the sheet: C3, R1, RESET1
Changed lines of the file:
@@
 F 0 "C1" H 4215 3446 50  0000 L CNN
 F 1 "0.1 uF" H 4215 3355 50  0000 L CNN
-F 2 "Capacitor_SMD:C_0603_1608Metric_Pad1.05x0.95mm_HandSolder" H 4138 3250 50  0001 C CNN
+F 2 "Capacitor_THT:CP_Radial_D4.0mm_P2.00mm" H 4138 3250 50  0001 C CNN
 F 3 "~" H 4100 3400 50  0001 C CNN
 F 4 "C271438" H 4100 3400 50  0001 C CNN "LCSC"
@@
 L power:GND #PWR0102
 U 1 1 619447C3
-P 4900 4050
-F 0 "#PWR0102" H 4900 3800 50  0001 C CNN
-F 1 "GND" H 4905 3877 50  0000 C CNN
-F 2 "" H 4900 4050 50  0001 C CNN
-F 3 "" H 4900 4050 50  0001 C CNN
-	1    4900 4050
+P 4750 4050
+F 0 "#PWR0102" H 4750 3800 50  0001 C CNN
+F 1 "GND" H 4755 3877 50  0000 C CNN
+F 2 "" H 4750 4050 50  0001 C CNN
+F 3 "" H 4750 4050 50  0001 C CNN
+	1    4750 4050
 	1    0    0    -1
 $EndComp
@@
 L Device:C C3
 U 1 1 619447C9
-P 4900 3400
-F 0 "C3" H 5015 3446 50  0000 L CNN
-F 1 "0.3 uF" H 5015 3355 50  0000 L CNN
-F 2 "Capacitor_SMD:C_0603_1608Metric_Pad1.05x0.95mm_HandSolder" H 4938 3250 50  0001 C CNN
-F 3 "~" H 4900 3400 50  0001 C CNN
-	1    4900 3400
+P 4900 3800
+F 0 "C3" H 5015 3846 50  0000 L CNN
+F 1 "0.3 uF" H 5015 3755 50  0000 L CNN
+F 2 "Capacitor_THT:CP_Radial_D5.0mm_P2.50mm" H 4938 3650 50  0001 C CNN
+F 3 "~" H 4900 3800 50  0001 C CNN
+	1    4900 3800
 	1    0    0    -1
 $EndComp
@@
 L Device:R R1
 U 1 1 619447CF
-P 4900 3900
-F 0 "R1" H 4970 3946 50  0000 L CNN
-F 1 "10k" H 4970 3855 50  0000 L CNN
-F 2 "Resistor_SMD:R_1206_3216Metric_Pad1.42x1.75mm_HandSolder" V 4830 3900 50  0001 C CNN
-F 3 "~" H 4900 3900 50  0001 C CNN
-F 4 "C17902" H 4900 3900 50  0001 C CNN "LCSC"
-	1    4900 3900
+P 4900 3400
+F 0 "R1" H 4970 3446 50  0000 L CNN
+F 1 "10k" H 4970 3355 50  0000 L CNN
+F 2 "Resistor_SMD:R_1206_3216Metric_Pad1.42x1.75mm_HandSolder" V 4830 3400 50  0001 C CNN
+F 3 "~" H 4900 3400 50  0001 C CNN
+F 4 "C17902" H 4900 3400 50  0001 C CNN "LCSC"
+	1    4900 3400
 	1    0    0    -1
 $EndComp
@@
 L Switch:SW_Push RESET1
 U 1 1 61944795
-P 4600 3400
-F 0 "RESET1" V 4646 3352 50  0000 R CNN
-F 1 "SW_Push" V 4555 3352 50  0000 R CNN
-F 2 "Button_Switch_THT:SW_PUSH_6mm" H 4600 3600 50  0001 C CNN
-F 3 "~" H 4600 3600 50  0001 C CNN
-	1    4600 3400
+P 4600 3800
+F 0 "RESET1" V 4646 3752 50  0000 R CNN
+F 1 "SW_Push" V 4555 3752 50  0000 R CNN
+F 2 "RC522:boton" H 4600 4000 50  0001 C CNN
+F 3 "~" H 4600 4000 50  0001 C CNN
+	1    4600 3800
 	0    -1   -1   0
 $EndComp
@@
 Connection ~ 4100 3150
 Wire Wire Line
-	4100 3150 4600 3150
-Wire Wire Line
 	3700 3250 3700 3150
 Connection ~ 3700 3150
@@
 Connection ~ 4900 3600
 Wire Wire Line
-	4900 3600 4900 3750
-Wire Wire Line
 	4900 3600 4600 3600
-Wire Wire Line
-	4600 3200 4600 3150
-Connection ~ 4600 3150
-Wire Wire Line
-	4600 3150 4900 3150
 Text HLabel 7750 4800 2    50   Input ~ 0
 BOOT
@@
 F 2 "Capacitor_SMD:C_0603_1608Metric_Pad1.05x0.95mm_HandSolder" H 5488 3200 50  0001 C CNN
 F 3 "~" H 5450 3350 50  0001 C CNN
-F 4 "C0603" H 5450 3350 50  0001 C CNN "LCSC"
+F 4 "C44567" H 5450 3350 50  0001 C CNN "LCSC"
 	1    5450 3350
 	1    0    0    -1
@@
 F 2 "LED_SMD:LED_0603_1608Metric_Pad1.05x0.95mm_HandSolder" H 4150 5500 50  0001 C CNN
 F 3 "~" H 4150 5500 50  0001 C CNN
-F 4 "C138547" V 4150 5500 50  0001 C CNN "LCSC"
+F 4 "C375447" V 4150 5500 50  0001 C CNN "LCSC"
 	1    4150 5500
 	0    -1   -1   0
@@
 	0    -1   -1   0
 $EndComp
+Wire Wire Line
+	4100 3150 4900 3150
+Wire Wire Line
+	4900 4000 4900 3950
+Wire Wire Line
+	4600 4000 4750 4000
+Wire Wire Line
+	4900 3650 4900 3600
+Wire Wire Line
+	4750 4000 4750 4050
+Connection ~ 4750 4000
+Wire Wire Line
+	4750 4000 4900 4000
 $EndSCHEMATC
