File: schematics/schematics/schematics.kicad_pcb (KiCad board)
At the start: 2 copper layers, 63.5 x 64.8 mm, 35 parts, among them J1 Conn_01x02, J2 Conn_01x03, J4 Conn_01x02, K1 SANYOU_SRD_Form_C, SW2 SW_Push, U1 ESP32-WROVER, U2 RC522, U3 AS608, U4 MT3608_PCB, U5 AMS1117

Commit message: .
Parts:
- removed J1, J4: Conn_01x02, Connector_JST:JST_EH_B2B-EH-A_1x02_P2.50mm_Vertical
- removed J2: Conn_01x03, Connector_PinHeader_2.00mm:PinHeader_1x03_P2.00mm_Vertical
- added  : , MountingHole:MountingHole_3mm, F.Cu at (150.1, 145.5)
- added  : , MountingHole:MountingHole_3mm, F.Cu at (87.6, 181.4)
- added  : , MountingHole:MountingHole_3mm, F.Cu at (87.6, 145.5)
- added  : , MountingHole:MountingHole_3mm, F.Cu at (150.1, 181.4)
- added BTR1: Conn_01x02, Connector_JST:JST_EH_B2B-EH-A_1x02_P2.50mm_Vertical, F.Cu at (87.6, 172.7)
- added C10: C, Capacitor_SMD:C_0603_1608Metric_Pad1.05x0.95mm_HandSolder, F.Cu at (115.5, 179.8)
- added C9: C, Capacitor_SMD:C_0603_1608Metric_Pad1.05x0.95mm_HandSolder, F.Cu at (107.8, 177.8)
- added Cerradura1: Conn_01x02, Connector_JST:JST_EH_B2B-EH-A_1x02_P2.50mm_Vertical, F.Cu at (140.7, 172.5)
- added D9: SS34, Diode_SMD:D_1206_3216Metric_Pad1.42x1.75mm_HandSolder, F.Cu at (120.9, 181.9)
- added L1: 22 uH, inductor:IND_RLS-226-R, F.Cu at (131.2, 180.3)
- added PRGMER1: Conn_01x03, Connector_PinHeader_2.00mm:PinHeader_1x03_P2.00mm_Vertical, F.Cu at (140.0, 179.6)
- added R10: 10k, Resistor_SMD:R_1206_3216Metric_Pad1.42x1.75mm_HandSolder, F.Cu at (95.0, 180.1)
- added R11: 62k, Resistor_SMD:R_1206_3216Metric_Pad1.42x1.75mm_HandSolder, F.Cu at (105.2, 181.4)
- added R12: 3.3k, Resistor_SMD:R_1206_3216Metric_Pad1.42x1.75mm_HandSolder, F.Cu at (110.2, 181.4)
- C4: value C -> 100 pF
- U2: footprint ESP32-WROVER-I:RC522 -> Connector_JST:JST_EH_B8B-EH-A_1x08_P2.50mm_Vertical
- U4: value MT3608_PCB -> MT3608; footprint mt3608:mt3608pcb -> mt3608:mt3608
- moved U2 116.5 mm to (150.4, 154.4)
- moved U3 115.7 mm to (87.6, 161.8), turned to 90 degrees
- moved D7 109.7 mm to (113.8, 160.6), turned to 90 degrees
- moved K1 107.6 mm to (101.1, 157.7)
- moved R2 96.8 mm to (124.0, 160.6), turned to 270 degrees
- moved R7 96.7 mm to (118.8, 160.5)
- moved D4 93.5 mm to (106.9, 144.6), turned to 90 degrees
- moved D5 93.3 mm to (106.9, 148.4), turned to 90 degrees
- moved D6 93.0 mm to (106.9, 152.3), turned to 90 degrees
- moved D1 92.6 mm to (94.0, 144.7), turned to 270 degrees
- moved D3 92.5 mm to (102.6, 144.6), turned to 270 degrees
- moved C8 91.2 mm to (114.0, 176.3), turned to 270 degrees
- moved U4 89.7 mm to (100.1, 180.1), turned to 180 degrees
- moved SW2 89.1 mm to (128.0, 170.9), turned to 0 degrees
- moved D2 88.3 mm to (98.3, 144.7), turned to 270 degrees
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Connections:
- U4 pad 1: /AS608/3v3 -> Net-(D9-Pad2)
- U4 pad 3: /Cerradura/12v -> Net-(R11-Pad2)
- U4 pad 4: GND -> Net-(R10-Pad1)
Routing:
- net GND: track 349.7 -> 176.6 mm, vias 2 -> 5
- net /Cerradura/CERRADURA: track 25.5 -> 74.2 mm, vias 0 -> 1
- net Net-(Cerradura1-Pad1): track 27.0 -> 74.1 mm
- net /AS608/3v3: track 162.0 -> 200.8 mm, vias 0 -> 2
- net /ESP32/RST: track 45.6 -> 9.96 mm
- net Net-(R3-Pad1): track 37.9 -> 4.31 mm, vias 2 -> 0
- net Net-(R4-Pad1): track 35.3 -> 4.93 mm, vias 2 -> 0
- net Net-(D1-Pad2): track 15.9 -> 45.4 mm, vias 0 -> 2
- net /Cerradura/12v: track 50.2 -> 79.0 mm, vias 0 -> 2
- net Net-(BTR1-Pad2): track 7.08 -> 35.7 mm
- net Net-(R5-Pad1): track 41.8 -> 17.6 mm, vias 2 -> 0
- net Net-(R2-Pad1): track 27.4 -> 4.55 mm, vias 2 -> 0
- net Net-(C3-Pad2): track 25.2 -> 44.1 mm
- net Net-(D9-Pad2): track 0.00 -> 18.5 mm
- net Net-(D2-Pad2): track 17.4 -> 35.0 mm, vias 0 -> 2
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- added copper zone on F.Cu, net GND
- removed copper zone on B.Cu, net GND
Other:
- board outline removed
- net class information added: clearance 0.3, trace_width 0.6, via_dia 0.7, via_drill 0.4
- net class power added: clearance 0.3, trace_width 0.6, via_dia 1.6, via_drill 0.5

Commit message: .
Parts:
- removed the   at (150.1, 145.5)
- removed the   at (87.6, 181.4)
- removed the   at (87.6, 145.5)
- removed the   at (150.1, 181.4)
- removed D10: 1N5406, Diode_SMD:D_1206_3216Metric_Pad1.42x1.75mm_HandSolder
- removed U1: ESP32-WROVER, ESP32-WROVER-I:XCVR_ESP32-WROVER-I
- added  : , MountingHole:MountingHole_3mm, F.Cu at (172.7, 120.4)
- added   : ESP32-WROVER, ESP32-WROVER-I:XCVR_ESP32-WROVER-I, F.Cu at (200.7, 126.2)
- added  : , MountingHole:MountingHole_3mm, F.Cu at (215.4, 120.4)
- added H1: , MountingHole:MountingHole_3mm, F.Cu at (215.1, 169.9)
- added H2: , MountingHole:MountingHole_3mm, F.Cu at (172.7, 169.9)
- C1: footprint Capacitor_SMD:C_0603_1608Metric_Pad1.05x0.95mm_HandSolder -> Capacitor_THT:CP_Radial_D4.0mm_P2.00mm
- C10, C9: value C -> 22 uF
- C3, C8: footprint Capacitor_SMD:C_0603_1608Metric_Pad1.05x0.95mm_HandSolder -> Capacitor_THT:CP_Radial_D5.0mm_P2.50mm
- D1: value LED -> On
- D2: value LED -> Wifi
- D3: value LED -> Open
- D4: value LED -> lvl1
- D5: value LED -> lvl2
- D6: value LED -> lvl3
- D7, D8: footprint Diode_SMD:D_1206_3216Metric_Pad1.42x1.75mm_HandSolder -> Diode_SMD:D_SOD-123
- D9: footprint Diode_SMD:D_1206_3216Metric_Pad1.42x1.75mm_HandSolder -> Diode_SMD:D_SMA
- PRGMER1: footprint Connector_PinHeader_2.00mm:PinHeader_1x03_P2.00mm_Vertical -> Connector_JST:JST_EH_B3B-EH-A_1x03_P2.50mm_Vertical
- RESET1, SW2: footprint Button_Switch_THT:SW_PUSH_6mm -> RC522:boton
- moved U3 127.5 mm to (214.9, 153.4)
- moved K1 107.7 mm to (208.8, 155.4), turned to 180 degrees
- moved D7 93.5 mm to (206.0, 144.8), turned to 0 degrees
- moved SW2 92.7 mm to (215.1, 139.2), turned to 90 degrees
- moved BTR1 92.5 mm to (180.1, 169.4), turned to 0 degrees
- moved PRGMER1 91.7 mm to (215.6, 127.8), turned to 270 degrees
- moved RESET1 88.1 mm to (178.6, 121.1), turned to 270 degrees
- moved R10 85.8 mm to (177.5, 156.7), turned to 0 degrees
- moved D8 84.5 mm to (197.6, 145.0), turned to 180 degrees
- moved R11 82.2 mm to (182.4, 153.1), turned to 270 degrees
- moved R12 82.2 mm to (187.5, 153.1), turned to 90 degrees
- moved U4 82.0 mm to (177.3, 152.4)
- moved D1 79.9 mm to (173.1, 133.9), turned to 0 degrees
- moved R1 76.4 mm to (184.2, 120.1)
- moved C7 76.1 mm to (189.9, 165.1), turned to 0 degrees
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Connections:
- C3 pad 1: /AS608/3v3 -> Net-(C3-Pad1)
- C3 pad 2: Net-(C3-Pad2) -> GND
- C8 pad 1: Net-(C8-Pad1) -> Net-(BTR1-Pad2)
- R1 pad 1: Net-(C3-Pad2) -> /AS608/3v3
- R1 pad 2: GND -> Net-(C3-Pad1)
- RESET1 pad 1: Net-(C3-Pad2) -> GND
- RESET1 pad 2: /AS608/3v3 -> Net-(C3-Pad1)
- U5 pad 3: Net-(C8-Pad1) -> Net-(BTR1-Pad2)
Routing:
- net GND: track 176.6 -> 121.1 mm, vias 5 -> 12
- net /ESP32/MISO: track 16.1 -> 70.1 mm, vias 0 -> 1
- net /Cerradura/CERRADURA: track 74.2 -> 25.9 mm
- net Net-(C3-Pad2): track 44.1 -> 0.00 mm
- net /ESP32/BOOT: track 49.6 -> 6.77 mm, vias 1 -> 0
- net /ESP32/RST: track 9.96 -> 51.1 mm
- net /ESP32/TX1: track 39.5 -> 9.15 mm, vias 1 -> 0
- net Net-(Cerradura1-Pad1): track 74.1 -> 44.0 mm
- net /ESP32/SCK: track 19.6 -> 48.0 mm, vias 0 -> 1
- net Net-(D1-Pad2): track 45.4 -> 17.6 mm, vias 2 -> 0
- net /ESP32/SDA: track 21.1 -> 47.4 mm, vias 0 -> 1
- net /ESP32/RX1: track 37.4 -> 11.5 mm, vias 1 -> 0
- net /ESP32/MOSI: track 33.1 -> 57.9 mm
- net Net-(C3-Pad1): track 0.00 -> 20.7 mm
- net Net-(BTR1-Pad2): track 35.7 -> 18.0 mm
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Other:
- board outline added: 50 x 56.6 mm
- net class 3V3 added: clearance 0.3, trace_width 0.4, via_dia 0.8, via_drill 0.4
