File: schematics/schematics/schematics.sch (KiCad schematic (older format))
At the start: 4 parts, among them J2 Conn_01x03, SW2 SW_Push

Commit message: .
Connections:
- net AS608/3v3: now also R8.1
Changed lines of the file:
@@
 F3 "CERRADURA" I L 5000 4850 50
-$EndSheet
-$Sheet
-S 2850 3400 650  800
-U 618F1C26
-F0 "Potencia" 50
-F1 "Potencia.sch" 50
 $EndSheet
 Wire Wire Line
@@
 Wire Wire Line
 	4850 2200 5000 2200
-Wire Wire Line
-	4850 3450 4850 2200
 Wire Wire Line
 	6500 3850 6450 3850
@@
 Wire Wire Line
 	4450 2650 4800 2650
+Wire Wire Line
+	3650 3050 3100 3050
+Wire Wire Line
+	3100 3050 3100 2200
+Wire Wire Line
+	3100 2200 4850 2200
+Wire Wire Line
+	4850 2200 4850 3450
+$Sheet
+S 2950 3750 550  300
+U 618F1C26
+F0 "Potencia" 50
+F1 "Potencia.sch" 50
+F2 "3v3" I R 3500 3850 50
+F3 "12v" I R 3500 3950 50
+$EndSheet
+Wire Wire Line
+	3650 3050 3650 3850
+Wire Wire Line
+	3500 3850 3650 3850
+Wire Wire Line
+	3650 3850 4000 3850
+Connection ~ 3650 3850
+Wire Wire Line
+	3500 3950 3700 3950
+Wire Wire Line
+	3700 3950 3700 5000
+Wire Wire Line
+	3700 5000 5000 5000
 $EndSCHEMATC

Commit message: .
Parts:
- added H1, H2, H3, H4: MountingHole, MountingHole:MountingHole_3mm, symbol Mechanical:MountingHole
- renumbered J2 to PRGMER1
Changed lines of the file:
@@
 $EndComp
 $Comp
-L Connector_Generic:Conn_01x03 J2
+L Connector_Generic:Conn_01x03 PRGMER1
 U 1 1 619D36FF
 P 3350 2750
-F 0 "J2" H 3268 2425 50  0000 C CNN
+F 0 "PRGMER1" H 3268 2425 50  0000 C CNN
 F 1 "Conn_01x03" H 3268 2516 50  0000 C CNN
 F 2 "Connector_PinHeader_2.00mm:PinHeader_1x03_P2.00mm_Vertical" H 3350 2750 50  0001 C CNN
@@
 Wire Wire Line
 	3700 5000 5000 5000
+$Comp
+L Mechanical:MountingHole H1
+U 1 1 61B467BB
+P 3000 5100
+F 0 "H1" H 3100 5146 50  0000 L CNN
+F 1 "MountingHole" H 3100 5055 50  0000 L CNN
+F 2 "MountingHole:MountingHole_3mm" H 3000 5100 50  0001 C CNN
+F 3 "~" H 3000 5100 50  0001 C CNN
+	1    3000 5100
+	1    0    0    -1
+$EndComp
+$Comp
+L Mechanical:MountingHole H2
+U 1 1 61B47007
+P 3000 5300
+F 0 "H2" H 3100 5346 50  0000 L CNN
+F 1 "MountingHole" H 3100 5255 50  0000 L CNN
+F 2 "MountingHole:MountingHole_3mm" H 3000 5300 50  0001 C CNN
+F 3 "~" H 3000 5300 50  0001 C CNN
+	1    3000 5300
+	1    0    0    -1
+$EndComp
+$Comp
+L Mechanical:MountingHole H3
+U 1 1 61B48122
+P 3000 5500
+F 0 "H3" H 3100 5546 50  0000 L CNN
+F 1 "MountingHole" H 3100 5455 50  0000 L CNN
+F 2 "MountingHole:MountingHole_3mm" H 3000 5500 50  0001 C CNN
+F 3 "~" H 3000 5500 50  0001 C CNN
+	1    3000 5500
+	1    0    0    -1
+$EndComp
+$Comp
+L Mechanical:MountingHole H4
+U 1 1 61B4930B
+P 3000 5700
+F 0 "H4" H 3100 5746 50  0000 L CNN
+F 1 "MountingHole" H 3100 5655 50  0000 L CNN
+F 2 "MountingHole:MountingHole_3mm" H 3000 5700 50  0001 C CNN
+F 3 "~" H 3000 5700 50  0001 C CNN
+	1    3000 5700
+	1    0    0    -1
+$EndComp
 $EndSCHEMATC

Commit message: .
Parts:
- R8, R9: LCSC (none) -> C247434
Changed lines of the file:
@@
 F 2 "Resistor_SMD:R_1206_3216Metric_Pad1.42x1.75mm_HandSolder" V 4430 4100 50  0001 C CNN
 F 3 "~" H 4500 4100 50  0001 C CNN
+F 4 "C247434" H 4500 4100 50  0001 C CNN "LCSC"
 	1    4500 4100
 	1    0    0    -1
@@
 F 2 "Resistor_SMD:R_1206_3216Metric_Pad1.42x1.75mm_HandSolder" V 4080 3850 50  0001 C CNN
 F 3 "~" H 4150 3850 50  0001 C CNN
+F 4 "C247434" V 4150 3850 50  0001 C CNN "LCSC"
 	1    4150 3850
 	0    -1   -1   0

Commit message: .
Parts:
- PRGMER1: footprint Connector_PinHeader_2.00mm:PinHeader_1x03_P2.00mm_Vertical -> Connector_JST:JST_EH_B3B-EH-A_1x03_P2.50mm_Vertical; LCSC (none) -> C144394
- SW2: footprint Button_Switch_THT:SW_PUSH_6mm -> RC522:boton; LCSC (none) -> C720477
Other:
- moved on the sheet: PRGMER1
Changed lines of the file:
@@
 F 0 "SW2" H 4250 2935 50  0000 C CNN
 F 1 "SW_Push" H 4250 2844 50  0000 C CNN
-F 2 "Button_Switch_THT:SW_PUSH_6mm" H 4250 2850 50  0001 C CNN
+F 2 "RC522:boton" H 4250 2850 50  0001 C CNN
 F 3 "~" H 4250 2850 50  0001 C CNN
+F 4 "C720477" H 4250 2650 50  0001 C CNN "LCSC"
 	1    4250 2650
 	1    0    0    -1
@@
 L Connector_Generic:Conn_01x03 PRGMER1
 U 1 1 619D36FF
-P 3350 2750
-F 0 "PRGMER1" H 3268 2425 50  0000 C CNN
-F 1 "Conn_01x03" H 3268 2516 50  0000 C CNN
-F 2 "Connector_PinHeader_2.00mm:PinHeader_1x03_P2.00mm_Vertical" H 3350 2750 50  0001 C CNN
-F 3 "~" H 3350 2750 50  0001 C CNN
-	1    3350 2750
+P 3300 2750
+F 0 "PRGMER1" H 3218 2425 50  0000 C CNN
+F 1 "Conn_01x03" H 3218 2516 50  0000 C CNN
+F 2 "Connector_JST:JST_EH_B3B-EH-A_1x03_P2.50mm_Vertical" H 3300 2750 50  0001 C CNN
+F 3 "~" H 3300 2750 50  0001 C CNN
+F 4 "C144394" H 3300 2750 50  0001 C CNN "LCSC"
+	1    3300 2750
 	-1   0    0    1
 $EndComp
@@
 Wire Wire Line
 	3900 2650 4050 2650
-Wire Wire Line
-	3550 2650 3900 2650
-Wire Wire Line
-	3550 2750 4750 2750
-Wire Wire Line
-	3550 2850 4650 2850
 Wire Wire Line
 	4650 3750 5000 3750
@@
 	1    0    0    -1
 $EndComp
+Wire Wire Line
+	3500 2650 3900 2650
+Wire Wire Line
+	3500 2750 4750 2750
+Wire Wire Line
+	3500 2850 4650 2850
 $EndSCHEMATC
